File: DNKR64/DNKR64.kicad_sch (KiCad schematic)
At the start: 160 parts, among them J1 SWD, J2 USB_C_Receptacle_USB2.0, Q1 AO3407, SW1 MX, SW10 MX, SW11 MX, SW12 MX, SW13 MX, SW14 MX, SW15 MX, SW16 MX, SW17 MX, SW18 MX, SW19 MX, SW2 MX, SW20 MX, SW21 MX, SW22 MX, SW23 MX, SW24 MX, SW25 MX, SW26 MX, SW27 MX, SW28 MX, SW29 MX, SW3 MX, SW30 MX, SW31 MX, SW32 MX, SW33 MX, SW34 MX, SW35 MX, SW36 MX, SW37 MX, SW38 MX, SW39 MX, SW4 MX, SW40 MX, SW41 MX, SW42 MX, SW43 MX, SW44 MX, SW45 MX, SW46 MX, SW47 MX, SW48 MX, SW49 MX, SW5 MX, SW50 MX, SW51 MX, SW52 MX, SW53 MX, SW54 MX, SW55 MX, SW56 MX, SW57 MX, SW58 MX, SW59 MX, SW6 MX, SW60 MX, SW61 MX, SW62 MX, SW63 MX, SW64 MX, SW65 MX, SW66 MX, SW67 MX, SW68 MX, SW7 MX, SW8 MX, SW9 MX, U1 HOLYIOT-18010, U2 DW01A, U3 FS8205, U4 MCP73831, U5 XC6220-3.3V

Commit message: Plot gerbers
Parts:
- removed D56, D68: 1N5819, symbol Device:D_Small
- removed SW56, SW68: MX, symbol Switch:SW_Push
- BT1: footprint (none) -> Ladniys-Lib:Connector_Battery_18650
- C1: footprint (none) -> Ladniys-Lib:C_0603
- D1, D10, D11, D12, D13, D14, D15, D16, D17, D18, D19, D2, D20, D21, D22, D23, D24, D25, D26, D27, D28, D29, D3, D30, D31, D32, D33, D34, D35, D36, D37, D38, D39, D4, D40, D41, D42, D43, D44, D45, D46, D47, D48, D49, D5, D50, D51, D52, D53, D54, D55, D6, D7, D8, D9: footprint (none) -> Ladniys-Lib:D_SOD-123
- D56: renamed from D57; footprint (none) -> Ladniys-Lib:D_SOD-123
- D57: renamed from D58; footprint (none) -> Ladniys-Lib:D_SOD-123
- D58: renamed from D59; footprint (none) -> Ladniys-Lib:D_SOD-123
- D59: renamed from D60; footprint (none) -> Ladniys-Lib:D_SOD-123
- D60: renamed from D61; footprint (none) -> Ladniys-Lib:D_SOD-123
- D61: renamed from D62; footprint (none) -> Ladniys-Lib:D_SOD-123
- D62: renamed from D63; footprint (none) -> Ladniys-Lib:D_SOD-123
- D63: renamed from D64; footprint (none) -> Ladniys-Lib:D_SOD-123
- D64: renamed from D65; footprint (none) -> Ladniys-Lib:D_SOD-123
- D65: renamed from D66; footprint (none) -> Ladniys-Lib:D_SOD-123
- D66: renamed from D67; footprint (none) -> Ladniys-Lib:D_SOD-123
- D67: renamed from D69; footprint TK44:LED_0603 -> Ladniys-Lib:LED_0603
- D68: renamed from D70; footprint TK44:D_SOD-123 -> Ladniys-Lib:D_SOD-123
- D69: renamed from D71; footprint TK44:LED_0603 -> Ladniys-Lib:LED_0603
- J1: footprint TK44:Connector_THT_1x4_2.54 -> Ladniys-Lib:Connector_THT_1x4_2.54
- J2: footprint TK44:USB-C-C168688 -> Ladniys-Lib:USB-C-C168688
- Q1: footprint TK44:SOT-23 -> Ladniys-Lib:SOT-23
- R1, R2: footprint (none) -> Ladniys-Lib:R_0603
- R10, R3, R4, R5, R6, R7, R8, R9: footprint TK44:R_0603 -> Ladniys-Lib:R_0603
- SW1, SW10, SW11, SW12, SW13, SW16, SW17, SW18, SW19, SW2, SW20, SW21, SW22, SW23, SW24, SW25, SW26, SW27, SW3, SW30, SW31, SW32, SW33, SW34, SW35, SW36, SW37, SW38, SW39, SW4, SW40, SW41, SW43, SW44, SW45, SW46, SW47, SW48, SW49, SW5, SW50, SW51, SW52, SW54, SW6, SW7, SW8, SW9: footprint (none) -> Ladniys-Lib:SW_Hotswap_MX_1.00u
- SW14: footprint (none) -> Ladniys-Lib:SW_Hotswap_MX_2.00u
- SW15, SW55: footprint (none) -> Ladniys-Lib:SW_Hotswap_MX_1.50u
- SW28: footprint (none) -> Ladniys-Lib:SW_Hotswap_MX_ISO
- SW29, SW53: footprint (none) -> Ladniys-Lib:SW_Hotswap_MX_1.75u
- SW42: footprint (none) -> Ladniys-Lib:SW_Hotswap_MX_2.25u
- SW56: renamed from SW57; footprint (none) -> Ladniys-Lib:SW_Hotswap_MX_1.00u
- SW57: renamed from SW58; footprint (none) -> Ladniys-Lib:SW_Hotswap_MX_1.00u
- SW58: renamed from SW59; footprint (none) -> Ladniys-Lib:SW_Hotswap_MX_1.25u
- SW59: renamed from SW60; footprint (none) -> Ladniys-Lib:SW_Hotswap_MX_2.75u_Reversed
- SW60: renamed from SW61; footprint (none) -> Ladniys-Lib:SW_Hotswap_MX_1.25u
- SW61: renamed from SW62; footprint (none) -> Ladniys-Lib:SW_Hotswap_MX_2.25u_Reversed
- SW62: renamed from SW63; footprint (none) -> Ladniys-Lib:SW_Hotswap_MX_1.00u
- SW63: renamed from SW64; footprint (none) -> Ladniys-Lib:SW_Hotswap_MX_1.00u
- SW64: renamed from SW65; footprint (none) -> Ladniys-Lib:SW_Hotswap_MX_1.00u
- SW65: renamed from SW66; footprint (none) -> Ladniys-Lib:SW_Hotswap_MX_1.00u
- SW66: renamed from SW67; footprint (none) -> Ladniys-Lib:SW_Hotswap_MX_1.00u
- SWT1: footprint TK44:K2-1187SQ -> Ladniys-Lib:K2-1187SQ
- U1: footprint TK44:Holyiot-18010-nRF52840 -> Ladniys-Lib:Holyiot-18010-nRF52840_mini
- U2, U3: footprint (none) -> Ladniys-Lib:SOT-23-6
- U4, U5: footprint TK44:SOT-23-5 -> Ladniys-Lib:SOT-23-5
Connections:
- net C1: now also SW55.2; no longer SW56.2
- net C12: now also SW64.2
- net C14: no longer SW55.2
- net C2: now also SW56.2; no longer SW57.2
- net C3: now also SW57.2; no longer SW58.2
- net C4: now also SW58.2; no longer SW59.2
- net C5: now also SW59.2; no longer SW60.2
- net C6: now also SW60.2; no longer SW61.2
- net C7: now also SW61.2; no longer SW62.2
- net C8: now also SW62.2; no longer SW63.2
- net C9: now also SW63.2; no longer SW64.2
- net R4: no longer D55.1 (K)
- net R5: now also D55.1 (K)
- net C15: no longer names the net of U1.29 (P1.01)
- no-connect marks 10 -> 11
Other:
- moved on the sheet: D55, D56, D57, D58, D59, D60, D61, D62, D63, D64, SW55, SW56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
